Commit message: adding base_footprint to base_link dynamic frame

File: husky_description/urdf/husky.urdf.xacro (robot description, xacro)
@@ -74,7 +74,7 @@
   <link name="base_footprint"/>
   <joint name="base_footprint_joint" type="fixed">
-    <origin xyz="0 0 ${wheel_vertical_offset - wheel_radius}" rpy="0 0 0" />
-    <parent link="base_link" />
-    <child link="base_footprint" />
+    <origin xyz="0 0 ${wheel_radius-wheel_vertical_offset}" rpy="0 0 0" />
+    <parent link="base_footprint" />
+    <child link="base_link" />
   </joint>
   <!-- Interial link stores the robot's inertial information -->
